File: PCB/vacSwitch/vacSwitch.sch (KiCad schematic (older format))
At the start: 28 parts, among them J1 Mains, J2 RS232, J3 ISP, J4 VoltFreeContact, K1 HE721A0510, Q1 BC547, U1 ATtiny85-20PU, U2 ACS712xLCTR-20A, U3 MOC3043M

Commit message: update PCB (errors fixed)
Parts:
- C4: footprint Capacitor_THT:CP_Radial_Tantal_D5.0mm_P2.50mm -> Capacitor_THT:CP_Radial_Tantal_D5.0mm_P5.00mm
Connections:
- net GND: no longer R3.2
- net VCC: now also K1.2, R3.2; no longer K1.6
- net at D6.1 (K), Q1.1 (C), U3.2: now also K1.6; no longer K1.2
Changed lines of the file:
@@
 F 0 "C4" H 3665 4196 50  0000 L CNN
 F 1 "10pF" H 3665 4105 50  0000 L CNN
-F 2 "Capacitor_THT:CP_Radial_Tantal_D5.0mm_P2.50mm" H 3588 4000 50  0001 C CNN
+F 2 "Capacitor_THT:CP_Radial_Tantal_D5.0mm_P5.00mm" H 3588 4000 50  0001 C CNN
 F 3 "~" H 3550 4150 50  0001 C CNN
 	1    3550 4150
@@
 Wire Wire Line
 	2650 2800 2650 2900
-Wire Wire Line
-	2650 2900 1850 2900
 Connection ~ 1850 2900
 $Comp
@@
 Connection ~ 6300 2500
 Wire Wire Line
-	6300 2500 6300 3550
-Connection ~ 6300 3550
-Wire Wire Line
-	6300 3550 6300 3750
-Wire Wire Line
 	6300 1500 6800 1500
 $Comp
 L power:VCC #PWR0101
 U 1 1 6182D683
-P 6700 2800
-F 0 "#PWR0101" H 6700 2650 50  0001 C CNN
-F 1 "VCC" H 6715 2973 50  0000 C CNN
-F 2 "" H 6700 2800 50  0001 C CNN
-F 3 "" H 6700 2800 50  0001 C CNN
-	1    6700 2800
+P 7050 4000
+F 0 "#PWR0101" H 7050 3850 50  0001 C CNN
+F 1 "VCC" H 7065 4173 50  0000 C CNN
+F 2 "" H 7050 4000 50  0001 C CNN
+F 3 "" H 7050 4000 50  0001 C CNN
+	1    7050 4000
 	1    0    0    -1
 $EndComp
@@
 Wire Wire Line
 	10050 1150 10650 1150
-Wire Wire Line
-	6300 3550 6700 3550
 Wire Wire Line
 	6700 2800 6700 2950
@@
 	2500 5850 2650 5850
 Connection ~ 2500 5850
+Wire Wire Line
+	6300 2500 6300 2800
+Wire Wire Line
+	6700 2800 6300 2800
+Connection ~ 6300 2800
+Wire Wire Line
+	6300 2800 6300 3750
+Wire Wire Line
+	6700 3550 6700 4000
+Wire Wire Line
+	6700 4000 7050 4000
+$Comp
+L power:VCC #PWR0102
+U 1 1 61B9555E
+P 2950 2900
+F 0 "#PWR0102" H 2950 2750 50  0001 C CNN
+F 1 "VCC" H 2965 3073 50  0000 C CNN
+F 2 "" H 2950 2900 50  0001 C CNN
+F 3 "" H 2950 2900 50  0001 C CNN
+	1    2950 2900
+	1    0    0    -1
+$EndComp
+Wire Wire Line
+	2650 2900 2950 2900
 $EndSCHEMATC

Commit message: Board updates. V1.1
Connections:
- net HOT: now also C6.2, D9.1 (A1), R11.2; no longer C6.1, D9.2 (A2), R12.2
- net VAC: now also C6.1, D9.2 (A2), R12.2; no longer C6.2, D9.1 (A1), R11.2
Changed lines of the file:
@@
 Wire Wire Line
 	8100 2900 7650 2900
+Text GLabel 9050 2900 2    50   Input ~ 0
+HOT
 Text GLabel 9050 2150 2    50   Input ~ 0
-HOT
-Text GLabel 9050 2900 2    50   Input ~ 0
 VAC
 Wire Wire Line
