File: PCB/vacSwitch/vacSwitch.kicad_pcb (KiCad board)
At the start: 2 copper layers, 91.2 x 50.8 mm, 28 parts, among them J1 Mains, J2 RS232, J3 ISP, J4 VoltFreeContact, K1 HE721A0510, Q1 BC547, U1 ATtiny85-20PU, U2 ACS712xLCTR-20A, U3 MOC3043M

Commit message: Board updates. V1.1
Parts:
- moved C6 16.6 mm to (130.8, 112.3), turned to 90 degrees
- moved R11 9.94 mm to (125.0, 96.5), turned to 180 degrees
- moved RV1 4.66 mm to (119.4, 100.6), turned to 0 degrees
- moved R12 0.28 mm to (124.2, 92.2)
Connections:
- C6 pad 1: HOT -> VAC
- C6 pad 2: VAC -> HOT
- D9 pad 1: VAC -> HOT
- D9 pad 2: HOT -> VAC
- R11 pad 2: VAC -> HOT
- R12 pad 2: HOT -> VAC
Routing:
- net VAC: track 40.7 -> 68.9 mm, vias 0 -> 1
- net Net-(D9-Pad3): track 31.8 -> 22.5 mm
- net NEUTRAL: track 42.8 -> 44.2 mm
- net HOT: track 46.7 -> 45.9 mm
- added copper zone on F.Cu, net HOT
- added copper zone on B.Cu, net NEUTRAL
- added copper zone on F.Cu, net VAC
Other:
- board text added: "GRB 2021 AutoSwitch V1.1"
- board text removed: "GRB 2021 AutoSwitch V1.0"

Commit message: Defaults tweak
Other:
- net class Default removed
